File: hardware/followsun-hardware.sch (KiCad schematic (older format))
At the start: 40 parts, among them J1 PowerSupply, J2 5V StepDown, J3 AzimuthSense, J4 ElevationSense, J5 Wind, J6 DS3231_Module, J7 AzimuthMotor, J8 ElevationMotor, K1 SANYOU_SRD_Form_C, K2 SANYOU_SRD_Form_C, K3 SANYOU_SRD_Form_C, K4 SANYOU_SRD_Form_C, SW1 WindMode, U1 LM4040DBZ-4.1, U2 ULN2803A

Commit message: v1.0
Other:
- note added: "wrong I2C pins !!"
Changed lines of the file:
@@
 Wire Wire Line
 	3050 7000 3300 7000
+Text Notes 5800 5800 0    50   ~ 0
+wrong I2C pins !!
 $EndSCHEMATC
